File: diploma.kicad_pcb (KiCad board)
At the start: 2 copper layers, 99.6 x 40.8 mm, 23 parts, among them J1 USB_B_Micro, J2 ICSP, U1 ATmega32U4-AU, Y1 Crystal_GND2

Commit message: - Cambio header de programacion por pads con via en el medio - Añado logo PCBWay para que nos patrocinen Bilbao
Parts:
- removed J2: ICSP, Connector_PinSocket_2.54mm:PinSocket_2x03_P2.54mm_Vertical
- added G***: LOGO, imagenes:logo PCBWay, B.Cu at (106.2, 87.2)
- added TP1: TestPoint, TestPoint:TestPoint_Pad_D1.5mm, B.Cu at (181.1, 70.4)
- added TP2: TestPoint, TestPoint:TestPoint_Pad_D1.5mm, B.Cu at (178.6, 70.4)
- added TP3: TestPoint, TestPoint:TestPoint_Pad_D1.5mm, B.Cu at (176.0, 70.4)
- added TP4: TestPoint, TestPoint:TestPoint_Pad_D1.5mm, B.Cu at (176.0, 72.9)
- added TP5: TestPoint, TestPoint:TestPoint_Pad_D1.5mm, B.Cu at (178.6, 73.0)
- added TP6: TestPoint, TestPoint:TestPoint_Pad_D1.5mm, B.Cu at (181.1, 73.0)
- BT2: footprint diploma_footprints:Pad_arrow_2_corto -> diploma_footprints:Pad_arrow_2_muy_corto
- moved G*** 2.00 mm to (112.0, 78.5)
Routing:
- net +5V: track 114.7 -> 111.9 mm, vias 0 -> 1
- net /MISO: track 40.5 -> 41.0 mm, vias 0 -> 1
- net /CLK: track 48.0 -> 48.4 mm, vias 0 -> 1
- net /reset: track 48.8 -> 48.6 mm, vias 0 -> 1
- net /MOSI: vias 1 -> 2
- net GND: vias 2 -> 8
Other:
- board text added: "Sponsored by"
